Commit message: [dynamixel_general_hw] mechanicalReduction must be considered in joint limits

File: dynamixel_general_hw/urdf/sample2.urdf (robot description, URDF)
Before this commit: robot sample_robot, 2 links, 1 joints
Joints:
- joint sample_joint: limit lower=-3.1415 upper=3.1415 effort=0 velocity=6.8 -> lower=-1.5707 upper=1.5707 effort=0 velocity=3.4
