Commit message: [dynamixel_general_hw] Add current-based position control and its sample

File: dynamixel_general_hw/urdf/sample6.urdf (robot description, URDF)
Before this commit: robot sample_robot, 2 links, 1 joints
Joints:
- joint sample_joint: limit effort=0 velocity=6.8 -> effort=0.92 velocity=6.8
